File: pcbs/hat/BatteryTester.kicad_pcb (KiCad board)
At the start: 2 copper layers, 146 parts, among them J1 Screw_Terminal_01x02, J2 XT60, J3 XT60, J4 XT60, J5 XT60, J6 XT60, J7 XT60, J8 XT60, J9 XT60, Q1 DMT6009LCT, Q10 AO3414, Q11 DMT6009LCT, Q12 AO3414, Q13 DMT6009LCT, Q14 AO3414, Q15 DMT6009LCT, Q16 AO3414, Q2 AO3414, Q3 DMT6009LCT, Q4 AO3414, Q5 DMT6009LCT, Q6 AO3414, Q7 DMT6009LCT, Q8 AO3414, Q9 DMT6009LCT, U1 INA181A2IDBVR, U10 TP5000_Breakout_Akaddy, U11 INA181A2IDBVR, U12 TP5000_Breakout_Akaddy, U13 INA181A2IDBVR, U14 TP5000_Breakout_Akaddy, U15 INA181A2IDBVR, U16 TP5000_Breakout_Akaddy, U17 NUCLEO-F401RE, U18 ADS7828, U19 ADS7828, U2 TP5000_Breakout_Akaddy, U20 ADS7828, U21 AP2138N-2.5TRG1, U22 LM3480-IM3-5.0, U23 SST25VF016B, U3 INA181A2IDBVR, U4 TP5000_Breakout_Akaddy, U5 INA181A2IDBVR, U6 TP5000_Breakout_Akaddy, U7 INA181A2IDBVR, U8 TP5000_Breakout_Akaddy, U9 INA181A2IDBVR

Commit message: beginning of the layout
Parts:
- removed the U22 at (65.4, 112.9)
- added C10: 1u, Capacitor_SMD:C_0805_2012Metric, F.Cu at (442.0, -48.3)
- added C13: optional, Capacitor_THT:CP_Radial_D6.3mm_P2.50mm, F.Cu at (475.0, -81.3)
- added C15: 1u, Capacitor_SMD:C_0805_2012Metric, F.Cu at (472.4, -48.3)
- added C18: optional, Capacitor_THT:CP_Radial_D6.3mm_P2.50mm, F.Cu at (505.5, -81.3)
- added C20: 1u, Capacitor_SMD:C_0805_2012Metric, F.Cu at (502.9, -48.3)
- added C23: optional, Capacitor_THT:CP_Radial_D6.3mm_P2.50mm, F.Cu at (475.0, 53.3)
- added C25: 1u, Capacitor_SMD:C_0805_2012Metric, F.Cu at (477.5, 20.3)
- added C28: optional, Capacitor_THT:CP_Radial_D6.3mm_P2.50mm, F.Cu at (444.5, 53.3)
- added C3: optional, Capacitor_THT:CP_Radial_D6.3mm_P2.50mm, F.Cu at (414.0, -81.3)
- added C30: 1u, Capacitor_SMD:C_0805_2012Metric, F.Cu at (447.0, 20.3)
- added C33: optional, Capacitor_THT:CP_Radial_D6.3mm_P2.50mm, F.Cu at (414.0, 53.3)
- added C35: 1u, Capacitor_SMD:C_0805_2012Metric, F.Cu at (416.6, 20.3)
- added C38: optional, Capacitor_THT:CP_Radial_D6.3mm_P2.50mm, F.Cu at (383.5, 53.3)
- added C40: 1u, Capacitor_SMD:C_0805_2012Metric, F.Cu at (386.1, 20.3)
- added C5: 1u, Capacitor_SMD:C_0805_2012Metric, F.Cu at (411.5, -48.3)
- added C8: optional, Capacitor_THT:CP_Radial_D6.3mm_P2.50mm, F.Cu at (444.5, -81.3)
- added SYM1: Courtyard for replication, CustomFootprints:replication_courtyard, F.Cu at (388.6, -94.0)
- added SYM2: Courtyard for replication, CustomFootprints:replication_courtyard, F.Cu at (419.1, -94.0)
- added SYM3: Courtyard for replication, CustomFootprints:replication_courtyard, F.Cu at (449.6, -94.0)
- added SYM4: Courtyard for replication, CustomFootprints:replication_courtyard, F.Cu at (480.1, -94.0)
- added SYM5: Courtyard for replication, CustomFootprints:replication_courtyard, F.Cu at (500.4, 66.0)
- added SYM6: Courtyard for replication, CustomFootprints:replication_courtyard, F.Cu at (469.9, 66.0)
- added SYM7: Courtyard for replication, CustomFootprints:replication_courtyard, F.Cu at (439.4, 66.0)
- added SYM8: Courtyard for replication, CustomFootprints:replication_courtyard, F.Cu at (408.9, 66.0)
- added U18: ADS7828, Package_SO:TSSOP-16_4.4x5mm_P0.65mm, F.Cu at (85.3, 116.1)
- C1, C11, C16, C21, C26, C31, C36, C6: value 200n -> 220n; footprint Capacitor_SMD:C_0603_1608Metric -> Capacitor_SMD:C_0805_2012Metric
- C42: renamed from C44; value 47u -> 100n; footprint Capacitor_SMD:C_1206_3216Metric -> Capacitor_SMD:C_0805_2012Metric
- C43: renamed from C46; value 22u -> 100n; footprint Capacitor_SMD:C_1206_3216Metric -> Capacitor_SMD:C_0805_2012Metric
- C44: renamed from C41; value 100n -> 47u; footprint Capacitor_SMD:C_0805_2012Metric -> Capacitor_SMD:C_1206_3216Metric
- C45: renamed from C42; value 100n -> 47u; footprint Capacitor_SMD:C_0805_2012Metric -> Capacitor_SMD:C_1206_3216Metric
- C46: renamed from C45; value 47u -> 22u
- J1: value Screw_Terminal_01x02 -> Supply Connector; footprint TerminalBlock:TerminalBlock_bornier-2_P5.08mm -> Connector_Phoenix_MSTB:PhoenixContact_MSTBA_2,5_2-G-5,08_1x02_P5.08mm_Horizontal
- J2, J3, J4, J5, J6, J7, J8, J9: value XT60 -> Battery Connector
- R1, R11, R12, R15, R18, R19, R22, R25, R26, R29, R32, R33, R36, R39, R4, R40, R43, R46, R47, R5, R50, R53, R54, R57, R58, R8: footprint Resistor_SMD:R_0603_1608Metric -> Resistor_SMD:R_0805_2012Metric
- U19: renamed from U23; value SST25VF016B -> ADS7828; footprint Package_SO:SOIC-8_5.275x5.275mm_P1.27mm -> Package_SO:TSSOP-16_4.4x5mm_P0.65mm
- U22: renamed from U19; value ADS7828 -> LM3480-5.0; footprint Package_SO:TSSOP-16_4.4x5mm_P0.65mm -> Package_TO_SOT_SMD:SOT-23
- U23: renamed from U20; value ADS7828 -> SST25VF016B; footprint Package_SO:TSSOP-16_4.4x5mm_P0.65mm -> Package_SO:SOIC-8_5.275x5.275mm_P1.27mm
- moved U9 382.6 mm to (491.5, 45.9), turned to -90 degrees
- moved C24 380.8 mm to (499.4, 45.7), turned to 90 degrees
- moved Q10 377.9 mm to (490.2, 30.5)
- moved U10 375.6 mm to (485.5, 40.0)
- moved R32 371.3 mm to (497.8, 43.2), turned to 180 degrees
- moved U6 369.7 mm to (464.5, -67.9), turned to 180 degrees
- moved U5 368.3 mm to (458.5, -73.8), turned to 90 degrees
- moved C11 365.2 mm to (473.4, -61.0)
- moved Q6 360.0 mm to (459.7, -58.4), turned to 180 degrees
- moved J4 356.8 mm to (467.4, -80.0), turned to 180 degrees
- moved C21 355.2 mm to (476.6, 33.0), turned to 180 degrees
- moved J6 353.8 mm to (482.6, 52.1)
- moved R30 352.6 mm to (485.1, 45.7), turned to -90 degrees
- moved C14 351.7 mm to (450.6, -73.7), turned to -90 degrees
- moved C22 349.5 mm to (495.3, 45.7), turned to 180 degrees
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- renumbered C48 to C41, C43 to C48, U18 to U20
Connections:
- C29 pad 2: /SENSOR_81 -> /SENSOR_61
- C39 pad 2: /SENSOR_61 -> /SENSOR_81
- C41 pad 1: GND -> +5V
- C41 pad 2: +3V3 -> GND
- C42 pad 1: GND -> +5V
- C42 pad 2: Net-(C44-Pad2) -> GND
- C43 pad 1: GND -> +5V
- C43 pad 2: Vref_I_SENS -> GND
- C44 pad 1: +5V -> GND
- C44 pad 2: GND -> Net-(C44-Pad2)
- C45 pad 1: +5V -> GND
- C45 pad 2: GND -> Net-(C45-Pad2)
- C46 pad 2: Net-(C45-Pad2) -> Vref_I_SENS
- C48 pad 1: +5V -> GND
- C48 pad 2: GND -> +3V3
- J2 pad 1: /SENSOR_10 -> /test-battery-1/GNDBAT
- J2 pad 2: /test-battery-1/GNDBAT -> /SENSOR_10
- J3 pad 1: /SENSOR_20 -> /test-battery-2/GNDBAT
- J3 pad 2: /test-battery-2/GNDBAT -> /SENSOR_20
- J4 pad 1: /SENSOR_30 -> /test-battery-3/GNDBAT
- J4 pad 2: /test-battery-3/GNDBAT -> /SENSOR_30
- J5 pad 1: /SENSOR_40 -> /test-battery-4/GNDBAT
- J5 pad 2: /test-battery-4/GNDBAT -> /SENSOR_40
- J6 pad 1: /SENSOR_50 -> /test-battery-5/GNDBAT
- J6 pad 2: /test-battery-5/GNDBAT -> /SENSOR_50
- J7 pad 1: /SENSOR_80 -> /test-battery-6/GNDBAT
- J7 pad 2: /test-battery-8/GNDBAT -> /SENSOR_60
- J8 pad 1: /SENSOR_70 -> /test-battery-7/GNDBAT
- J8 pad 2: /test-battery-7/GNDBAT -> /SENSOR_70
- J9 pad 1: /SENSOR_60 -> /test-battery-8/GNDBAT
- J9 pad 2: /test-battery-6/GNDBAT -> /SENSOR_80
- Q11 pad 2: /SENSOR_80 -> /SENSOR_60
- Q15 pad 2: /SENSOR_60 -> /SENSOR_80
- R36 pad 1: /SIGNAL_81 -> /SIGNAL_61
- R37 pad 1: /test-battery-8/GNDBAT -> /test-battery-6/GNDBAT
- R39 pad 2: /SENSOR_81 -> /SENSOR_61
- R40 pad 1: /SIGNAL_80 -> /SIGNAL_60
- R41 pad 1: /SENSOR_82 -> /SENSOR_62
- R50 pad 1: /SIGNAL_61 -> /SIGNAL_81
- R51 pad 1: /test-battery-6/GNDBAT -> /test-battery-8/GNDBAT
- R53 pad 2: /SENSOR_61 -> /SENSOR_81
- R54 pad 1: /SIGNAL_60 -> /SIGNAL_80
- R55 pad 1: /SENSOR_62 -> /SENSOR_82
- TH6 pad 2: /SENSOR_82 -> /SENSOR_62
- TH8 pad 2: /SENSOR_62 -> /SENSOR_82
- U12 pad 11: /SENSOR_83 -> /SENSOR_63
- U12 pad 3: /SENSOR_80 -> /SENSOR_60
- U16 pad 11: /SENSOR_63 -> /SENSOR_83
- U16 pad 3: /SENSOR_60 -> /SENSOR_80
- U19 pad 1: /Board/~{MEM_CE} -> /SENSOR_81
- U19 pad 2: /Board/MEM_MISO -> /SENSOR_71
- U19 pad 3: +3V3 -> /SENSOR_61
- U19 pad 4: GND -> /SENSOR_51
- U19 pad 5: /Board/MEM_MOSI -> /SENSOR_41
- U19 pad 6: /Board/MEM_SCK -> /SENSOR_31
- U19 pad 7: +3V3 -> /SENSOR_21
- U19 pad 8: +3V3 -> /SENSOR_11
- U20 pad 1: /SENSOR_10 -> /SENSOR_82
- U20 pad 13: GND -> +5V
- U20 pad 2: /SENSOR_20 -> /SENSOR_72
- U20 pad 3: /SENSOR_30 -> /SENSOR_62
- U20 pad 4: /SENSOR_40 -> /SENSOR_52
- U20 pad 5: /SENSOR_50 -> /SENSOR_42
- U20 pad 6: /SENSOR_60 -> /SENSOR_32
- U20 pad 7: /SENSOR_70 -> /SENSOR_22
- U20 pad 8: /SENSOR_80 -> /SENSOR_12
- U21 pad 1: Net-(C44-Pad2) -> GND
- U21 pad 3: GND -> Net-(C44-Pad2)
- U22 pad 1: /SENSOR_11 -> /Converters/ADC_Ref
- U22 pad 2: /SENSOR_21 -> Net-(C45-Pad2)
- U22 pad 3: /SENSOR_31 -> GND
- U23 pad 1: /SENSOR_12 -> /Board/~{MEM_CE}
- U23 pad 2: /SENSOR_22 -> /Board/MEM_MISO
- U23 pad 3: /SENSOR_32 -> +3V3
- U23 pad 4: /SENSOR_42 -> GND
- U23 pad 5: /SENSOR_52 -> /Board/MEM_MOSI
- U23 pad 6: /SENSOR_62 -> /Board/MEM_SCK
- U23 pad 7: /SENSOR_72 -> +3V3
- U23 pad 8: /SENSOR_82 -> +3V3
Routing:
- net Vref_I_SENS: vias 0 -> 15
- net (no net): vias 0 -> 1
Other:
- copper layers 2 -> 4

Commit message: wip
Parts:
- removed SYM1, SYM2, SYM3, SYM4, SYM5, SYM6, SYM7, SYM8: Courtyard for replication, CustomFootprints:replication_courtyard
- moved U19 344.5 mm to (365.8, -20.3), turned to 180 degrees
- moved U20 339.8 mm to (365.8, -12.7)
- moved U18 315.2 mm to (365.8, -27.9), turned to 180 degrees
- moved J1 300.4 mm to (332.7, 26.7)
- moved C41 294.0 mm to (323.3, -24.1)
- moved C43 294.0 mm to (318.2, -28.4)
- moved C44 294.0 mm to (328.2, -27.5)
- moved C47 294.0 mm to (318.2, -31.7)
- moved C48 294.0 mm to (327.7, -24.1)
- moved R57 294.0 mm to (332.0, -24.7)
- moved R58 294.0 mm to (332.4, -27.7)
- moved C42 294.0 mm to (323.9, -31.7)
- moved C45 294.0 mm to (333.8, -31.9)
- moved C46 294.0 mm to (318.2, -25.0)
- moved U22 287.7 mm to (325.1, -38.1)
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Connections:
- U17 pad CN10_1: /SENSOR_43 -> unconnected-(U17-PadCN10_1)
- U17 pad CN10_12: unconnected-(U17-PadCN10_12) -> /SIGNAL_10
- U17 pad CN10_13: /SIGNAL_11 -> unconnected-(U17-PadCN10_13)
- U17 pad CN10_14: /SIGNAL_81 -> /SIGNAL_21
- U17 pad CN10_15: /SIGNAL_21 -> unconnected-(U17-PadCN10_15)
- U17 pad CN10_16: /SENSOR_53 -> /SIGNAL_20
- U17 pad CN10_17: /SIGNAL_30 -> unconnected-(U17-PadCN10_17)
- U17 pad CN10_19: /SENSOR_23 -> unconnected-(U17-PadCN10_19)
- U17 pad CN10_2: /SENSOR_33 -> /SENSOR_13
- U17 pad CN10_21: /SIGNAL_61 -> unconnected-(U17-PadCN10_21)
- U17 pad CN10_23: /SIGNAL_51 -> unconnected-(U17-PadCN10_23)
- U17 pad CN10_24: /SIGNAL_41 -> unconnected-(U17-PadCN10_24)
- U17 pad CN10_25: /Board/MEM_SCK -> unconnected-(U17-PadCN10_25)
- U17 pad CN10_26: /SENSOR_83 -> unconnected-(U17-PadCN10_26)
- U17 pad CN10_27: /SIGNAL_20 -> unconnected-(U17-PadCN10_27)
- U17 pad CN10_28: /SENSOR_73 -> unconnected-(U17-PadCN10_28)
- U17 pad CN10_29: /SIGNAL_40 -> unconnected-(U17-PadCN10_29)
- U17 pad CN10_30: /SENSOR_63 -> unconnected-(U17-PadCN10_30)
- U17 pad CN10_33: /SIGNAL_71 -> unconnected-(U17-PadCN10_33)
- U17 pad CN10_4: /SENSOR_13 -> /SIGNAL_11
- U17 pad CN10_6: unconnected-(U17-PadCN10_6) -> /SENSOR_23
- U17 pad CN7_1: /SIGNAL_60 -> /Board/MEM_SCK
- U17 pad CN7_17: /SIGNAL_80 -> unconnected-(U17-PadCN7_17)
- U17 pad CN7_2: /SIGNAL_50 -> /Board/MEM_MISO
- U17 pad CN7_21: /SIGNAL_10 -> unconnected-(U17-PadCN7_21)
- U17 pad CN7_3: /SIGNAL_70 -> /Board/MEM_MOSI
- U17 pad CN7_34: /SIGNAL_31 -> unconnected-(U17-PadCN7_34)
- U17 pad CN7_35: /Board/MEM_MISO -> unconnected-(U17-PadCN7_35)
- U17 pad CN7_36: /Board/~{MEM_CE} -> unconnected-(U17-PadCN7_36)
- U17 pad CN7_37: /Board/MEM_MOSI -> unconnected-(U17-PadCN7_37)
- U17 pad CN7_4: unconnected-(U17-PadCN7_4) -> /Board/~{MEM_CE}
Routing:
- net (no net): track 0.00 -> 173.4 mm
- net /SIGNAL_41: track 0.00 -> 155.5 mm, vias 0 -> 1
- net /SENSOR_43: track 0.00 -> 129.9 mm
- net /SIGNAL_40: track 0.00 -> 129.7 mm, vias 0 -> 1
- net /SIGNAL_31: track 0.00 -> 109.3 mm, vias 0 -> 1
- net /SIGNAL_21: track 0.00 -> 107.8 mm, vias 0 -> 1
- net /SENSOR_23: track 0.00 -> 94.8 mm
- net /SENSOR_33: track 0.00 -> 90.4 mm
- net /SIGNAL_11: track 0.00 -> 88.0 mm, vias 0 -> 1
- net /SIGNAL_30: track 0.00 -> 87.2 mm, vias 0 -> 1
- net /SIGNAL_20: track 0.00 -> 83.7 mm, vias 0 -> 1
- net /SENSOR_13: track 0.00 -> 64.5 mm
- net /SENSOR_10: track 0.00 -> 58.6 mm
- net /SIGNAL_10: track 0.00 -> 58.1 mm, vias 0 -> 1
- net /SENSOR_11: track 0.00 -> 50.3 mm
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
Commit message: wip
Connections:
- U17 pad CN10_14: /SIGNAL_21 -> unconnected-(U17-PadCN10_14)
- U17 pad CN10_2: /SENSOR_13 -> /SIGNAL_11
- U17 pad CN10_24: unconnected-(U17-PadCN10_24) -> /SIGNAL_21
- U17 pad CN10_27: unconnected-(U17-PadCN10_27) -> /SIGNAL_41
- U17 pad CN10_28: unconnected-(U17-PadCN10_28) -> /SIGNAL_40
- U17 pad CN10_29: unconnected-(U17-PadCN10_29) -> /SENSOR_43
- U17 pad CN10_30: unconnected-(U17-PadCN10_30) -> /SIGNAL_30
- U17 pad CN10_33: unconnected-(U17-PadCN10_33) -> /SIGNAL_31
- U17 pad CN10_34: unconnected-(U17-PadCN10_34) -> /SENSOR_33
- U17 pad CN10_4: /SIGNAL_11 -> /SENSOR_13
Routing:
- net /SIGNAL_21: track 107.8 -> 94.7 mm
- net /SENSOR_33: track 90.4 -> 99.3 mm
- net /SIGNAL_40: track 129.7 -> 138.7 mm
- net /SIGNAL_11: track 88.0 -> 80.1 mm
- net /SIGNAL_41: track 155.5 -> 162.7 mm
- net /SENSOR_13: track 64.5 -> 58.0 mm
- net /SENSOR_43: track 129.9 -> 136.3 mm
- net /SIGNAL_31: track 109.3 -> 111.8 mm
- net /SIGNAL_30: track 87.2 -> 89.7 mm

Commit message: finish the pin assignment
Connections:
- U17 pad CN10_17: unconnected-(U17-PadCN10_17) -> /SIGNAL_61
- U17 pad CN10_19: unconnected-(U17-PadCN10_19) -> /SIGNAL_60
- U17 pad CN10_2: /SIGNAL_11 -> /SENSOR_13
- U17 pad CN10_20: Net-(U17-PadCN10_20) -> GND
- U17 pad CN10_21: unconnected-(U17-PadCN10_21) -> /SENSOR_63
- U17 pad CN10_22: unconnected-(U17-PadCN10_22) -> /SIGNAL_51
- U17 pad CN10_23: unconnected-(U17-PadCN10_23) -> /SIGNAL_50
- U17 pad CN10_25: unconnected-(U17-PadCN10_25) -> /SENSOR_53
- U17 pad CN10_30: /SIGNAL_30 -> /SIGNAL_31
- U17 pad CN10_33: /SIGNAL_31 -> /SIGNAL_30
- U17 pad CN10_4: /SENSOR_13 -> /SIGNAL_11
- U17 pad CN10_9: Net-(U17-PadCN10_20) -> GND
- U17 pad CN7_28: unconnected-(U17-PadCN7_28) -> /SIGNAL_81
- U17 pad CN7_30: unconnected-(U17-PadCN7_30) -> /SIGNAL_71
- U17 pad CN7_35: unconnected-(U17-PadCN7_35) -> /SIGNAL_80
- U17 pad CN7_36: unconnected-(U17-PadCN7_36) -> /SENSOR_73
- U17 pad CN7_37: unconnected-(U17-PadCN7_37) -> /SENSOR_83
- U17 pad CN7_38: unconnected-(U17-PadCN7_38) -> /SIGNAL_70
Routing:
- net /SENSOR_53: track 0.00 -> 185.7 mm
- net /SIGNAL_51: track 0.00 -> 179.4 mm, vias 0 -> 1
- net /SIGNAL_50: track 0.00 -> 176.9 mm, vias 0 -> 1
- net /SENSOR_63: track 0.00 -> 166.5 mm
- net /SIGNAL_60: track 0.00 -> 156.4 mm, vias 0 -> 1
- net /SIGNAL_61: track 0.00 -> 149.1 mm, vias 0 -> 1
- net /SENSOR_73: track 0.00 -> 90.8 mm
- net /SIGNAL_70: track 0.00 -> 75.0 mm, vias 0 -> 1
- net /SIGNAL_71: track 0.00 -> 72.0 mm, vias 0 -> 1
- net /SENSOR_83: track 0.00 -> 67.1 mm
- net /SIGNAL_80: track 0.00 -> 58.6 mm, vias 0 -> 1
- net /SIGNAL_81: track 0.00 -> 34.8 mm, vias 0 -> 1
- net /SIGNAL_31: track 111.8 -> 121.8 mm
- net /SIGNAL_11: track 80.1 -> 87.7 mm
- net /SENSOR_13: track 58.0 -> 64.5 mm
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