File: pcbs/hat/test-battery.kicad_sch (KiCad schematic)
At the start: 18 parts, among them J2 XT60, Q1 Q_NMOS_DGS, Q2 Q_NMOS_DGS, U1 INA181A2IDBVR, U2 TP5000_Breakout_Akaddy

Commit message: add memory + check footprints
Parts:
- removed C3: 0u, symbol Device:C
- removed Q1: Q_NMOS_DGS, Package_TO_SOT_THT:TO-220-3_Vertical, symbol Device:Q_NMOS_DGS
- removed Q2: Q_NMOS_DGS, Package_TO_SOT_SMD:SOT-223, symbol Device:Q_NMOS_DGS
- added C3: optional, Capacitor_THT:CP_Radial_D6.3mm_P2.50mm, symbol Device:C_Polarized
- added Q1: DMT6009LCT, Package_TO_SOT_THT:TO-220-3_Vertical, symbol Device:Q_NMOS_GDS
- added Q2: AO3414, Package_TO_SOT_SMD:SOT-23, symbol Device:Q_NMOS_GDS
- C1: value 200n -> 220n; footprint Capacitor_SMD:C_0603_1608Metric -> Capacitor_SMD:C_0805_2012Metric
- C2: footprint Capacitor_SMD:C_0603_1608Metric -> Capacitor_SMD:C_0805_2012Metric
- C5: footprint (none) -> Capacitor_SMD:C_0805_2012Metric
- J2: value XT60 -> Battery Connector
- R1, R4, R5: footprint Resistor_SMD:R_0603_1608Metric -> Resistor_SMD:R_0805_2012Metric
Connections:
- net GND: now also C3.2, Q1.3 (S), Q2.3 (S)
- net V_SENS: now also C3.1, Q1.2 (D)
- net at C1.1, R1.2, R3.1: now also Q1.1 (G)
- net at R5.2, R7.1: now also Q2.1 (G)
- net at U2.2 (GND), U2.4 (GND): now also Q2.2 (D)
Other:
- note added: "The mosfet can handle about 12A without cooling. For the vacuum chamber we maybe should think about some cooling. Maybe those will help?"
- note added: "There should be relativly low current flow via the GND-Pin, so a small transisotr should be fine here."
- note removed: "Battery Connector"
Changed lines of the file:
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@@
+    (effects (font (size 1.27 1.27)) (justify left bottom))
+  )
+  (text "There should be relativly low current flow via the\nGND-Pin, so a small transisotr should be fine here."
+    (at 186.055 149.86 0)
     (effects (font (size 1.27 1.27)) (justify left bottom))
   )
@@
     (effects (font (size 1.27 1.27)) (justify left bottom))
   )
-  (text "Battery Connector" (at 39.37 31.75 0)
+  (text "The mosfet can handle about 12A without cooling.\nFor the vacuum chamber we maybe should think about\nsome cooling. Maybe those will help?"
+    (at 74.295 133.985 0)
     (effects (font (size 1.27 1.27)) (justify left bottom))
   )
@@
     (effects (font (size 1.27 1.27)) (justify right))
   )
+  (symbol (lib_id "Device:Q_NMOS_GDS") (at 67.31 114.3 0) (unit 1)
+    (in_bom yes) (on_board yes) (fields_autoplaced)
+    (property "Reference" "Q1" (id 0) (at 73.66 113.0299 0)
+      (effects (font (size 1.27 1.27)) (justify left))
+    )
+    (property "Value" "DMT6009LCT" (id 1) (at 73.66 115.5699 0)
+      (effects (font (size 1.27 1.27)) (justify left))
+    )
+    (property "Footprint" "Package_TO_SOT_THT:TO-220-3_Vertical" (id 2) (at 72.39 111.76 0)
+      (effects (font (size 1.27 1.27)) hide)
+    )
+    (property "Datasheet" "https://www.mouser.at/ProductDetail/Diodes-Incorporated/DMT6009LCT?qs=rN85NNvew%2FSKNXyjWLi4%2Fw%3D%3D" (id 3) (at 67.31 114.3 0)
+      (effects (font (size 1.27 1.27)) hide)
+    )
+    (pin "1")
+    (pin "2")
+    (pin "3")
+  )
   (symbol (lib_id "power:+5V") (at 88.265 38.735 0) (unit 1)
     (in_bom yes) (on_board yes) (fields_autoplaced)
@@
       (effects (font (size 1.27 1.27)) (justify left))
     )
-    (property "Value" "200n" (id 1) (at 49.53 124.4599 0)
-      (effects (font (size 1.27 1.27)) (justify left))
-    )
-    (property "Footprint" "Capacitor_SMD:C_0603_1608Metric" (id 2) (at 46.6852 127 0)
+    (property "Value" "220n" (id 1) (at 49.53 124.4599 0)
+      (effects (font (size 1.27 1.27)) (justify left))
+    )
+    (property "Footprint" "Capacitor_SMD:C_0805_2012Metric" (id 2) (at 46.6852 127 0)
       (effects (font (size 1.27 1.27)) hide)
     )
@@
     (pin "4")
   )
-  (symbol (lib_id "Device:C") (at 107.95 111.76 0) (unit 1)
-    (in_bom yes) (on_board yes) (fields_autoplaced)
-    (property "Reference" "C3" (id 0) (at 111.125 110.4899 0)
-      (effects (font (size 1.27 1.27)) (justify left))
-    )
-    (property "Value" "0u" (id 1) (at 111.125 113.0299 0)
-      (effects (font (size 1.27 1.27)) (justify left))
-    )
-    (property "Footprint" "" (id 2) (at 108.9152 115.57 0)
-      (effects (font (size 1.27 1.27)) hide)
-    )
-    (property "Datasheet" "~" (id 3) (at 107.95 111.76 0)
-      (effects (font (size 1.27 1.27)) hide)
-    )
-    (pin "1")
-    (pin "2")
-  )
   (symbol (lib_id "Device:R") (at 117.475 57.15 90) (unit 1)
     (in_bom yes) (on_board yes) (fields_autoplaced)
     (property "Reference" "R4" (id 0) (at 117.475 50.8 90))
     (property "Value" "1k" (id 1) (at 117.475 53.34 90))
-    (property "Footprint" "Resistor_SMD:R_0603_1608Metric" (id 2) (at 117.475 58.928 90)
+    (property "Footprint" "Resistor_SMD:R_0805_2012Metric" (id 2) (at 117.475 58.928 90)
       (effects (font (size 1.27 1.27)) hide)
     )
@@
     (pin "1")
   )
+  (symbol (lib_id "Device:Q_NMOS_GDS") (at 179.705 139.7 0) (unit 1)
+    (in_bom yes) (on_board yes) (fields_autoplaced)
+    (property "Reference" "Q2" (id 0) (at 186.055 138.4299 0)
+      (effects (font (size 1.27 1.27)) (justify left))
+    )
+    (property "Value" "AO3414" (id 1) (at 186.055 140.9699 0)
+      (effects (font (size 1.27 1.27)) (justify left))
+    )
+    (property "Footprint" "Package_TO_SOT_SMD:SOT-23" (id 2) (at 184.785 137.16 0)
+      (effects (font (size 1.27 1.27)) hide)
+    )
+    (property "Datasheet" "https://media.digikey.com/pdf/Data%20Sheets/Alpha%20&%20Omega/AO3414.pdf" (id 3) (at 179.705 139.7 0)
+      (effects (font (size 1.27 1.27)) hide)
+    )
+    (pin "1")
+    (pin "2")
+    (pin "3")
+  )
   (symbol (lib_id "power:GND") (at 69.85 129.54 0) (unit 1)
     (in_bom yes) (on_board yes) (fields_autoplaced)
@@
     (property "Reference" "R1" (id 0) (at 35.56 107.95 90))
     (property "Value" "680" (id 1) (at 35.56 110.49 90))
-    (property "Footprint" "Resistor_SMD:R_0603_1608Metric" (id 2) (at 35.56 116.078 90)
+    (property "Footprint" "Resistor_SMD:R_0805_2012Metric" (id 2) (at 35.56 116.078 90)
       (effects (font (size 1.27 1.27)) hide)
     )
@@
   (symbol (lib_id "STS_Other:Link") (at 207.645 128.27 0) (unit 1)
     (in_bom yes) (on_board yes) (fields_autoplaced)
-    (property "Reference" "#Z1" (id 0) (at 207.645 124.714 0)
+    (property "Reference" "#Z2" (id 0) (at 207.645 124.714 0)
       (effects (font (size 1.27 1.27)) hide)
     )
@@
     (pin "1")
   )
+  (symbol (lib_id "STS_Other:Link") (at 114.935 135.89 0) (unit 1)
+    (in_bom yes) (on_board yes) (fields_autoplaced)
+    (property "Reference" "#Z1" (id 0) (at 114.935 132.334 0)
+      (effects (font (size 1.27 1.27)) hide)
+    )
+    (property "Value" "Link" (id 1) (at 116.205 132.334 0)
+      (effects (font (size 1.27 1.27)) (justify right) hide)
+    )
+    (property "Footprint" "" (id 2) (at 112.395 133.604 0)
+      (effects (font (size 1.27 1.27)) hide)
+    )
+    (property "Datasheet" "https://www.amazon.de/WayinTop-Unterlegscheibe-MOSFET-Transistor-Spannungsregler-20mmx15mmx10mm/dp/B081GS15N6/ref=sr_1_1_sspa?crid=31TSACA9W33GA&keywords=to220+k%C3%BChlk%C3%B6rper&qid=1663520226&sprefix=tos22%2Caps%2C91&sr=8-1-spons&psc=1" (id 3) (at 112.395 133.604 0)
+      (effects (font (size 1.27 1.27)) hide)
+    )
+  )
   (symbol (lib_id "Device:R_Shunt") (at 50.8 57.15 0) (unit 1)
     (in_bom yes) (on_board yes)
@@
     (pin "4")
   )
-  (symbol (lib_id "Device:Q_NMOS_DGS") (at 179.705 139.7 0) (unit 1)
-    (in_bom yes) (on_board yes) (fields_autoplaced)
-    (property "Reference" "Q2" (id 0) (at 186.055 138.4299 0)
-      (effects (font (size 1.27 1.27)) (justify left))
-    )
-    (property "Value" "Q_NMOS_DGS" (id 1) (at 186.055 140.9699 0)
-      (effects (font (size 1.27 1.27)) (justify left))
-    )
-    (property "Footprint" "Package_TO_SOT_SMD:SOT-223" (id 2) (at 184.785 137.16 0)
-      (effects (font (size 1.27 1.27)) hide)
-    )
-    (property "Datasheet" "~" (id 3) (at 179.705 139.7 0)
-      (effects (font (size 1.27 1.27)) hide)
-    )
-    (pin "1")
-    (pin "2")
-    (pin "3")
-  )
   (symbol (lib_id "power:GND") (at 45.72 129.54 0) (unit 1)
     (in_bom yes) (on_board yes) (fields_autoplaced)
@@
     (pin "2")
   )
+  (symbol (lib_id "Device:C_Polarized") (at 107.95 111.76 0) (unit 1)
+    (in_bom yes) (on_board yes) (fields_autoplaced)
+    (property "Reference" "C3" (id 0) (at 111.125 109.6009 0)
+      (effects (font (size 1.27 1.27)) (justify left))
+    )
+    (property "Value" "optional" (id 1) (at 111.125 112.1409 0)
+      (effects (font (size 1.27 1.27)) (justify left))
+    )
+    (property "Footprint" "Capacitor_THT:CP_Radial_D6.3mm_P2.50mm" (id 2) (at 108.9152 115.57 0)
+      (effects (font (size 1.27 1.27)) hide)
+    )
+    (property "Datasheet" "~" (id 3) (at 107.95 111.76 0)
+      (effects (font (size 1.27 1.27)) hide)
+    )
+    (pin "1")
+    (pin "2")
+  )
   (symbol (lib_id "STS_Other:Link") (at 207.645 132.08 0) (unit 1)
     (in_bom yes) (on_board yes) (fields_autoplaced)
-    (property "Reference" "#Z2" (id 0) (at 207.645 128.524 0)
+    (property "Reference" "#Z3" (id 0) (at 207.645 128.524 0)
       (effects (font (size 1.27 1.27)) hide)
     )
@@
     (property "Reference" "C2" (id 0) (at 81.915 38.1 90))
     (property "Value" "100n" (id 1) (at 81.915 40.64 90))
-    (property "Footprint" "Capacitor_SMD:C_0603_1608Metric" (id 2) (at 85.725 44.7548 0)
+    (property "Footprint" "Capacitor_SMD:C_0805_2012Metric" (id 2) (at 85.725 44.7548 0)
       (effects (font (size 1.27 1.27)) hide)
     )
@@
     (in_bom yes) (on_board yes)
     (property "Reference" "J2" (id 0) (at 39.37 35.56 0))
-    (property "Value" "XT60" (id 1) (at 38.1 37.465 0))
+    (property "Value" "Battery Connector" (id 1) (at 31.75 37.465 0))
     (property "Footprint" "Connector_Phoenix_MSTB:PhoenixContact_MSTBA_2,5_2-G-5,08_1x02_P5.08mm_Horizontal" (id 2) (at 43.18 35.56 0)
       (effects (font (size 1.27 1.27)) hide)
@@
     (property "Reference" "R5" (id 0) (at 161.925 133.35 90))
     (property "Value" "680" (id 1) (at 161.925 135.89 90))
-    (property "Footprint" "Resistor_SMD:R_0603_1608Metric" (id 2) (at 161.925 141.478 90)
+    (property "Footprint" "Resistor_SMD:R_0805_2012Metric" (id 2) (at 161.925 141.478 90)
       (effects (font (size 1.27 1.27)) hide)
     )
@@
     (pin "1")
     (pin "2")
-  )
-  (symbol (lib_id "Device:Q_NMOS_DGS") (at 67.31 114.3 0) (unit 1)
-    (in_bom yes) (on_board yes)
-    (property "Reference" "Q1" (id 0) (at 73.66 113.0299 0)
-      (effects (font (size 1.27 1.27)) (justify left))
-    )
-    (property "Value" "Q_NMOS_DGS" (id 1) (at 73.66 115.5699 0)
-      (effects (font (size 1.27 1.27)) (justify left))
-    )
-    (property "Footprint" "Package_TO_SOT_THT:TO-220-3_Vertical" (id 2) (at 72.39 111.76 0)
-      (effects (font (size 1.27 1.27)) hide)
-    )
-    (property "Datasheet" "~" (id 3) (at 67.31 114.3 0)
-      (effects (font (size 1.27 1.27)) hide)
-    )
-    (pin "1")
-    (pin "2")
-    (pin "3")
   )
   (symbol (lib_id "Device:R") (at 167.64 55.88 0) (unit 1)
@@
       (effects (font (size 1.27 1.27)) (justify left))
     )
-    (property "Footprint" "" (id 2) (at 180.0352 59.69 0)
-      (effects (font (size 1.27 1.27)) hide)
-    )
+    (property "Footprint" "Capacitor_SMD:C_0805_2012Metric" (id 2) (at 180.0352 59.69 0)
+      (effects (font (size 1.27 1.27)) hide)
+    )

Commit message: beginning of the layout
Parts:
- added SYM1: Courtyard for replication, CustomFootprints:replication_courtyard, symbol Graphic:SYM_Magnet_Large
Connections:
- net GNDBAT: now also J2.1 (Pin_1); no longer J2.2 (Pin_2)
- net V_SENS: now also J2.2 (Pin_2); no longer J2.1 (Pin_1)
Other:
- moved on the sheet: J2
Changed lines of the file:
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@@
     (pin "4")
+  )
+  (symbol (lib_id "Graphic:SYM_Magnet_Large") (at 31.115 157.48 0) (unit 1)
+    (in_bom yes) (on_board yes) (fields_autoplaced)
+    (property "Reference" "SYM1" (id 0) (at 31.115 152.4 0))
+    (property "Value" "Courtyard for replication" (id 1) (at 31.115 163.83 0))
+    (property "Footprint" "CustomFootprints:replication_courtyard" (id 2) (at 31.115 162.56 0)
+      (effects (font (size 1.27 1.27)) hide)
+    )
+    (property "Datasheet" "~" (id 3) (at 31.877 162.56 0)
+      (effects (font (size 1.27 1.27)) hide)
+    )
   )
   (symbol (lib_id "power:GND") (at 45.72 129.54 0) (unit 1)
@@
     (pin "2")
   )
-  (symbol (lib_id "Connector:Conn_01x02_Female") (at 43.18 35.56 0) (mirror y) (unit 1)
+  (symbol (lib_id "Connector:Conn_01x02_Female") (at 43.18 38.1 180) (unit 1)
     (in_bom yes) (on_board yes)
-    (property "Reference" "J2" (id 0) (at 39.37 35.56 0))
+    (property "Reference" "J2" (id 0) (at 39.37 34.925 0))
     (property "Value" "Battery Connector" (id 1) (at 31.75 37.465 0))
-    (property "Footprint" "Connector_Phoenix_MSTB:PhoenixContact_MSTBA_2,5_2-G-5,08_1x02_P5.08mm_Horizontal" (id 2) (at 43.18 35.56 0)
+    (property "Footprint" "Connector_Phoenix_MSTB:PhoenixContact_MSTBA_2,5_2-G-5,08_1x02_P5.08mm_Horizontal" (id 2) (at 43.18 38.1 0)
       (effects (font (size 1.27 1.27)) hide)
     )
-    (property "Datasheet" "~" (id 3) (at 43.18 35.56 0)
+    (property "Datasheet" "~" (id 3) (at 43.18 38.1 0)
       (effects (font (size 1.27 1.27)) hide)
     )

Commit message: wip
Parts:
- removed SYM1: Courtyard for replication, CustomFootprints:replication_courtyard, symbol Graphic:SYM_Magnet_Large
Changed lines of the file:
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@@
     (pin "4")
-  )
-  (symbol (lib_id "Graphic:SYM_Magnet_Large") (at 31.115 157.48 0) (unit 1)
-    (in_bom yes) (on_board yes) (fields_autoplaced)
-    (property "Reference" "SYM1" (id 0) (at 31.115 152.4 0))
-    (property "Value" "Courtyard for replication" (id 1) (at 31.115 163.83 0))
-    (property "Footprint" "CustomFootprints:replication_courtyard" (id 2) (at 31.115 162.56 0)
-      (effects (font (size 1.27 1.27)) hide)
-    )
-    (property "Datasheet" "~" (id 3) (at 31.877 162.56 0)
-      (effects (font (size 1.27 1.27)) hide)
-    )
   )
   (symbol (lib_id "power:GND") (at 45.72 129.54 0) (unit 1)

Commit message: reassign adc's
Connections:
- net GND: now also R2.1; no longer R2.4
- net GNDBAT: now also J2.2 (Pin_2), R2.4; no longer J2.1 (Pin_1), R2.1
- net V_SENS: now also J2.1 (Pin_1); no longer J2.2 (Pin_2)
Other:
- moved on the sheet: J2
Changed lines of the file:
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@@
+    (stroke (width 0) (type default) (color 0 0 0 0))
+  )
+  (wire (pts (xy 69.215 59.69) (xy 83.185 59.69))
     (stroke (width 0) (type default) (color 0 0 0 0))
   )
@@
     (stroke (width 0) (type default) (color 0 0 0 0))
   )
-  (wire (pts (xy 54.61 54.61) (xy 83.185 54.61))
+  (wire (pts (xy 64.135 54.61) (xy 69.215 59.69))
     (stroke (width 0) (type default) (color 0 0 0 0))
   )
@@
     (stroke (width 0) (type default) (color 0 0 0 0))
   )
+  (wire (pts (xy 54.61 59.69) (xy 64.135 59.69))
+    (stroke (width 0) (type default) (color 0 0 0 0))
+  )
   (polyline (pts (xy 147.32 81.28) (xy 147.32 12.7))
     (stroke (width 0) (type default) (color 0 0 0 0))
@@
     (stroke (width 0) (type default) (color 0 0 0 0))
   )
-  (wire (pts (xy 54.61 59.69) (xy 83.185 59.69))
-    (stroke (width 0) (type default) (color 0 0 0 0))
-  )
   (polyline (pts (xy 133.985 83.82) (xy 251.46 83.82))
     (stroke (width 0) (type default) (color 0 0 0 0))
@@
     (stroke (width 0) (type default) (color 0 0 0 0))
   )
+  (wire (pts (xy 69.215 54.61) (xy 83.185 54.61))
+    (stroke (width 0) (type default) (color 0 0 0 0))
+  )
   (wire (pts (xy 167.64 36.83) (xy 167.64 39.37))
     (stroke (width 0) (type default) (color 0 0 0 0))
@@
     (stroke (width 0) (type default) (color 0 0 0 0))
   )
+  (wire (pts (xy 54.61 54.61) (xy 64.135 54.61))
+    (stroke (width 0) (type default) (color 0 0 0 0))
+  )
   (wire (pts (xy 182.245 130.81) (xy 183.515 130.81))
     (stroke (width 0) (type default) (color 0 0 0 0))
@@
   )
   (wire (pts (xy 179.07 49.53) (xy 185.42 49.53))
+    (stroke (width 0) (type default) (color 0 0 0 0))
+  )
+  (wire (pts (xy 69.215 54.61) (xy 64.135 59.69))
     (stroke (width 0) (type default) (color 0 0 0 0))
   )
@@
     )
   )
-  (symbol (lib_id "Device:R_Shunt") (at 50.8 57.15 0) (unit 1)
+  (symbol (lib_id "Device:R_Shunt") (at 50.8 57.15 0) (mirror x) (unit 1)
     (in_bom yes) (on_board yes)
-    (property "Reference" "R2" (id 0) (at 48.26 55.88 0)
+    (property "Reference" "R2" (id 0) (at 47.625 55.88 0)
       (effects (font (size 1.27 1.27)) (justify right))
     )
-    (property "Value" "CST0612-FC-R005E (5mΩ)" (id 1) (at 48.26 58.42 0)
+    (property "Value" "CST0612-FC-R005E (5mΩ)" (id 1) (at 47.625 58.42 0)
       (effects (font (size 1.27 1.27)) (justify right))
     )
@@
     (pin "2")
   )
-  (symbol (lib_id "Connector:Conn_01x02_Female") (at 43.18 38.1 180) (unit 1)
+  (symbol (lib_id "Connector:Conn_01x02_Female") (at 43.18 35.56 0) (mirror y) (unit 1)
     (in_bom yes) (on_board yes)
-    (property "Reference" "J2" (id 0) (at 39.37 34.925 0))
+    (property "Reference" "J2" (id 0) (at 39.37 35.56 0))
     (property "Value" "Battery Connector" (id 1) (at 31.75 37.465 0))
-    (property "Footprint" "Connector_Phoenix_MSTB:PhoenixContact_MSTBA_2,5_2-G-5,08_1x02_P5.08mm_Horizontal" (id 2) (at 43.18 38.1 0)
-      (effects (font (size 1.27 1.27)) hide)
-    )
-    (property "Datasheet" "~" (id 3) (at 43.18 38.1 0)
-      (effects (font (size 1.27 1.27)) hide)
-    )
+    (property "Footprint" "Connector_Phoenix_MSTB:PhoenixContact_MSTBA_2,5_2-G-5,08_1x02_P5.08mm_Horizontal" (id 2) (at 43.18 35.56 0)
+      (effects (font (size 1.27 1.27)) hide)
+    )
+    (property "Datasheet" "~" (id 3) (at 43.18 35.56 0)
+      (effects (font (size 1.27 1.27)) hide)
+    )
